File: Hardware/InkTime_Schematic.brd (EAGLE design)
At the start: 46 x 35 mm, 105 parts, among them IC1 BQ25180YBGR, IC3 BMA421, IC4 DRV2605YZFR, IC9 RT6160AWSC, J1 503480-2400, J2 TC2030-IDC, J4 KH-TYPE-C-16P, Q1 20V/4.2A/52mΩ/1.4W, Q3 SI1308EDL-T1-GE3, U1 NRF52840_QF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

Commit message: update
Signed-off-by: Andreea21Radu <radu21andreea@yahoo.com>
Parts:
- C23, C27, C34, C42: device InkTime_v5:GRM011R60J152KE01L_2_CAPC0201X13N -> InkTime_v5:ERA-1AEB3401C_0201
- moved C19 1.70 mm to (34.6, 17.6)
- moved R7 0.36 mm to (34.9, 7.47)
- moved C38 0.19 mm to (20.5, 21.4)
Routing:
- net P0.14: track 9.03 -> 55.9 mm, vias 0 -> 2
- net EPD_RST: track 0.00 -> 32.2 mm, vias 0 -> 2
- net EPD_CS: track 0.00 -> 29.7 mm, vias 0 -> 2
- net GND: track 141.0 -> 169.6 mm, vias 13 -> 19
- net EPD_DC: track 0.00 -> 27.8 mm, vias 0 -> 2
- net MOSI: track 0.00 -> 25.0 mm, vias 0 -> 2
- net PMIC_INT: track 0.00 -> 17.9 mm, vias 0 -> 2
- net IMU_INT2: track 0.00 -> 13.4 mm, vias 0 -> 2
- net SDA: track 53.7 -> 59.8 mm, vias 8 -> 9
- net N$96: track 11.0 -> 14.7 mm
- net SCK: track 26.9 -> 26.3 mm
- net SCL: track 68.7 -> 68.9 mm, vias 4 -> 5
